Commit message: working on drivig robot

File: src/model_description/urdf/model.xacro (robot description, xacro)
@@ -20,5 +20,5 @@
     <origin xyz="0 0 0" rpy="0 0 0"/>
     <geometry>
-      <mesh filename="file://$(find model_description)/meshes/base_link.stl" scale="0.001 0.001 0.001"/>
+      <mesh filename="$(find model_description)/meshes/base_link.stl" scale="0.001 0.001 0.001"/>
     </geometry>
     <material name="silver"/>
@@ -27,5 +27,5 @@
     <origin xyz="0 0 0" rpy="0 0 0"/>
     <geometry>
-      <mesh filename="file://$(find model_description)/meshes/base_link.stl" scale="0.001 0.001 0.001"/>
+      <mesh filename="$(find model_description)/meshes/base_link.stl" scale="0.001 0.001 0.001"/>
     </geometry>
   </collision>
@@ -40,5 +40,5 @@
     <origin xyz="-0.05 0.256 -1.99" rpy="0 0 0"/>
     <geometry>
-      <mesh filename="file://$(find model_description)/meshes/stacker_slider_1.stl" scale="0.001 0.001 0.001"/>
+      <mesh filename="$(find model_description)/meshes/stacker_slider_1.stl" scale="0.001 0.001 0.001"/>
     </geometry>
     <material name="silver"/>
@@ -47,5 +47,5 @@
     <origin xyz="-0.05 0.256 -1.99" rpy="0 0 0"/>
     <geometry>
-      <mesh filename="file://$(find model_description)/meshes/stacker_slider_1.stl" scale="0.001 0.001 0.001"/>
+      <mesh filename="$(find model_description)/meshes/stacker_slider_1.stl" scale="0.001 0.001 0.001"/>
     </geometry>
   </collision>
@@ -60,5 +60,5 @@
     <origin xyz="-0.125 0.375 -0.49" rpy="0 0 0"/>
     <geometry>
-      <mesh filename="file://$(find model_description)/meshes/stacker_fork_1.stl" scale="0.001 0.001 0.001"/>
+      <mesh filename="$(find model_description)/meshes/stacker_fork_1.stl" scale="0.001 0.001 0.001"/>
     </geometry>
     <material name="silver"/>
@@ -67,5 +67,5 @@
     <origin xyz="-0.125 0.375 -0.49" rpy="0 0 0"/>
     <geometry>
-      <mesh filename="file://$(find model_description)/meshes/stacker_fork_1.stl" scale="0.001 0.001 0.001"/>
+      <mesh filename="$(find model_description)/meshes/stacker_fork_1.stl" scale="0.001 0.001 0.001"/>
     </geometry>
   </collision>
@@ -80,5 +80,5 @@
     <origin xyz="0.265391 0.32 -0.265" rpy="0 0 0"/>
     <geometry>
-      <mesh filename="file://$(find model_description)/meshes/r_caster_1.stl" scale="0.001 0.001 0.001"/>
+      <mesh filename="$(find model_description)/meshes/r_caster_1.stl" scale="0.001 0.001 0.001"/>
     </geometry>
     <material name="silver"/>
@@ -87,5 +87,5 @@
     <origin xyz="0.265391 0.32 -0.265" rpy="0 0 0"/>
     <geometry>
-      <mesh filename="file://$(find model_description)/meshes/r_caster_1.stl" scale="0.001 0.001 0.001"/>
+      <mesh filename="$(find model_description)/meshes/r_caster_1.stl" scale="0.001 0.001 0.001"/>
     </geometry>
   </collision>
@@ -100,5 +100,5 @@
     <origin xyz="0.27 -0.32 -0.265" rpy="0 0 0"/>
     <geometry>
-      <mesh filename="file://$(find model_description)/meshes/l_caster_1.stl" scale="0.001 0.001 0.001"/>
+      <mesh filename="$(find model_description)/meshes/l_caster_1.stl" scale="0.001 0.001 0.001"/>
     </geometry>
     <material name="silver"/>
@@ -107,5 +107,5 @@
     <origin xyz="0.27 -0.32 -0.265" rpy="0 0 0"/>
     <geometry>
-      <mesh filename="file://$(find model_description)/meshes/l_caster_1.stl" scale="0.001 0.001 0.001"/>
+      <mesh filename="$(find model_description)/meshes/l_caster_1.stl" scale="0.001 0.001 0.001"/>
     </geometry>
   </collision>
@@ -120,5 +120,5 @@
     <origin xyz="0.275391 0.35 -0.08" rpy="0 0 0"/>
     <geometry>
-      <mesh filename="file://$(find model_description)/meshes/r_caster_wheel_1.stl" scale="0.001 0.001 0.001"/>
+      <mesh filename="$(find model_description)/meshes/r_caster_wheel_1.stl" scale="0.001 0.001 0.001"/>
     </geometry>
     <material name="silver"/>
@@ -127,5 +127,5 @@
     <origin xyz="0.275391 0.35 -0.08" rpy="0 0 0"/>
     <geometry>
-      <mesh filename="file://$(find model_description)/meshes/r_caster_wheel_1.stl" scale="0.001 0.001 0.001"/>
+      <mesh filename="$(find model_description)/meshes/r_caster_wheel_1.stl" scale="0.001 0.001 0.001"/>
     </geometry>
   </collision>
@@ -140,5 +140,5 @@
     <origin xyz="0.28 -0.29 -0.08" rpy="0 0 0"/>
     <geometry>
-      <mesh filename="file://$(find model_description)/meshes/l_caster_wheel_1.stl" scale="0.001 0.001 0.001"/>
+      <mesh filename="$(find model_description)/meshes/l_caster_wheel_1.stl" scale="0.001 0.001 0.001"/>
     </geometry>
     <material name="silver"/>
@@ -147,5 +147,5 @@
     <origin xyz="0.28 -0.29 -0.08" rpy="0 0 0"/>
     <geometry>
-      <mesh filename="file://$(find model_description)/meshes/l_caster_wheel_1.stl" scale="0.001 0.001 0.001"/>
+      <mesh filename="$(find model_description)/meshes/l_caster_wheel_1.stl" scale="0.001 0.001 0.001"/>
     </geometry>
   </collision>
@@ -160,5 +160,5 @@
     <origin xyz="-1.14 0.34 -0.027" rpy="0 0 0"/>
     <geometry>
-      <mesh filename="file://$(find model_description)/meshes/r_static_wheel_1.stl" scale="0.001 0.001 0.001"/>
+      <mesh filename="$(find model_description)/meshes/r_static_wheel_1.stl" scale="0.001 0.001 0.001"/>
     </geometry>
     <material name="silver"/>
@@ -167,5 +167,5 @@
     <origin xyz="-1.14 0.34 -0.027" rpy="0 0 0"/>
     <geometry>
-      <mesh filename="file://$(find model_description)/meshes/r_static_wheel_1.stl" scale="0.001 0.001 0.001"/>
+      <mesh filename="$(find model_description)/meshes/r_static_wheel_1.stl" scale="0.001 0.001 0.001"/>
     </geometry>
   </collision>
@@ -180,5 +180,5 @@
     <origin xyz="-1.14 -0.34 -0.027" rpy="0 0 0"/>
     <geometry>
-      <mesh filename="file://$(find model_description)/meshes/l_static_wheel_1.stl" scale="0.001 0.001 0.001"/>
+      <mesh filename="$(find model_description)/meshes/l_static_wheel_1.stl" scale="0.001 0.001 0.001"/>
     </geometry>
     <material name="silver"/>
@@ -187,5 +187,5 @@
     <origin xyz="-1.14 -0.34 -0.027" rpy="0 0 0"/>
     <geometry>
-      <mesh filename="file://$(find model_description)/meshes/l_static_wheel_1.stl" scale="0.001 0.001 0.001"/>
+      <mesh filename="$(find model_description)/meshes/l_static_wheel_1.stl" scale="0.001 0.001 0.001"/>
     </geometry>
   </collision>
@@ -200,5 +200,5 @@
     <origin xyz="0.05 -0.29 -1.035" rpy="0 0 0"/>
     <geometry>
-      <mesh filename="file://$(find model_description)/meshes/steer_head_1.stl" scale="0.001 0.001 0.001"/>
+      <mesh filename="$(find model_description)/meshes/steer_head_1.stl" scale="0.001 0.001 0.001"/>
     </geometry>
     <material name="silver"/>
@@ -207,5 +207,5 @@
     <origin xyz="0.05 -0.29 -1.035" rpy="0 0 0"/>
     <geometry>
-      <mesh filename="file://$(find model_description)/meshes/steer_head_1.stl" scale="0.001 0.001 0.001"/>
+      <mesh filename="$(find model_description)/meshes/steer_head_1.stl" scale="0.001 0.001 0.001"/>
     </geometry>
   </collision>
@@ -220,5 +220,5 @@
     <origin xyz="0.902 0.345 -0.225194" rpy="0 0 0"/>
     <geometry>
-      <mesh filename="file://$(find model_description)/meshes/l_wheel_1.stl" scale="0.001 0.001 0.001"/>
+      <mesh filename="$(find model_description)/meshes/l_wheel_1.stl" scale="0.001 0.001 0.001"/>
     </geometry>
     <material name="silver"/>
@@ -227,5 +227,5 @@
     <origin xyz="0.902 0.345 -0.225194" rpy="0 0 0"/>
     <geometry>
-      <mesh filename="file://$(find model_description)/meshes/l_wheel_1.stl" scale="0.001 0.001 0.001"/>
+      <mesh filename="$(find model_description)/meshes/l_wheel_1.stl" scale="0.001 0.001 0.001"/>
     </geometry>
   </collision>
@@ -240,5 +240,5 @@
     <origin xyz="0.902 -0.345 -0.225194" rpy="0 0 0"/>
     <geometry>
-      <mesh filename="file://$(find model_description)/meshes/r_wheel_1.stl" scale="0.001 0.001 0.001"/>
+      <mesh filename="$(find model_description)/meshes/r_wheel_1.stl" scale="0.001 0.001 0.001"/>
     </geometry>
     <material name="silver"/>
@@ -247,5 +247,5 @@
     <origin xyz="0.902 -0.345 -0.225194" rpy="0 0 0"/>
     <geometry>
-      <mesh filename="file://$(find model_description)/meshes/r_wheel_1.stl" scale="0.001 0.001 0.001"/>
+      <mesh filename="$(find model_description)/meshes/r_wheel_1.stl" scale="0.001 0.001 0.001"/>
     </geometry>
   </collision>
@@ -260,5 +260,5 @@
     <origin xyz="0.902 -0.0 -0.533053" rpy="0 0 0"/>
     <geometry>
-      <mesh filename="file://$(find model_description)/meshes/steering_1.stl" scale="0.001 0.001 0.001"/>
+      <mesh filename="$(find model_description)/meshes/steering_1.stl" scale="0.001 0.001 0.001"/>
     </geometry>
     <material name="silver"/>
@@ -267,5 +267,5 @@
     <origin xyz="0.902 -0.0 -0.533053" rpy="0 0 0"/>
     <geometry>
-      <mesh filename="file://$(find model_description)/meshes/steering_1.stl" scale="0.001 0.001 0.001"/>
+      <mesh filename="$(find model_description)/meshes/steering_1.stl" scale="0.001 0.001 0.001"/>
     </geometry>
   </collision>

Commit message: problem with kinematic

File: src/model_description/urdf/model.xacro (robot description, xacro)
@@ -20,14 +20,14 @@
     <origin xyz="0 0 0" rpy="0 0 0"/>
     <geometry>
-      <mesh filename="$(find model_description)/meshes/base_link.stl" scale="0.001 0.001 0.001"/>
-    </geometry>
-    <material name="silver"/>
-  </visual>
-  <collision>
+      <mesh filename="package://model_description/meshes/base_link.stl" scale="0.001 0.001 0.001"/>
+    </geometry>
+    <material name="silver"/>
+  </visual>
+  <!-- <collision>
     <origin xyz="0 0 0" rpy="0 0 0"/>
     <geometry>
-      <mesh filename="$(find model_description)/meshes/base_link.stl" scale="0.001 0.001 0.001"/>
-    </geometry>
-  </collision>
+      <mesh filename="package://model_description/meshes/base_link.stl" scale="0.001 0.001 0.001"/>
+    </geometry>
+  </collision> -->
 </link>
 <link name="stacker_slider_1">
@@ -40,5 +40,5 @@
     <origin xyz="-0.05 0.256 -1.99" rpy="0 0 0"/>
     <geometry>
-      <mesh filename="$(find model_description)/meshes/stacker_slider_1.stl" scale="0.001 0.001 0.001"/>
+      <mesh filename="package://model_description/meshes/stacker_slider_1.stl" scale="0.001 0.001 0.001"/>
     </geometry>
     <material name="silver"/>
@@ -47,5 +47,5 @@
     <origin xyz="-0.05 0.256 -1.99" rpy="0 0 0"/>
     <geometry>
-      <mesh filename="$(find model_description)/meshes/stacker_slider_1.stl" scale="0.001 0.001 0.001"/>
+      <mesh filename="package://model_description/meshes/stacker_slider_1.stl" scale="0.001 0.001 0.001"/>
     </geometry>
   </collision>
@@ -60,5 +60,5 @@
     <origin xyz="-0.125 0.375 -0.49" rpy="0 0 0"/>
     <geometry>
-      <mesh filename="$(find model_description)/meshes/stacker_fork_1.stl" scale="0.001 0.001 0.001"/>
+      <mesh filename="package://model_description/meshes/stacker_fork_1.stl" scale="0.001 0.001 0.001"/>
     </geometry>
     <material name="silver"/>
@@ -67,5 +67,5 @@
     <origin xyz="-0.125 0.375 -0.49" rpy="0 0 0"/>
     <geometry>
-      <mesh filename="$(find model_description)/meshes/stacker_fork_1.stl" scale="0.001 0.001 0.001"/>
+      <mesh filename="package://model_description/meshes/stacker_fork_1.stl" scale="0.001 0.001 0.001"/>
     </geometry>
   </collision>
@@ -80,5 +80,5 @@
     <origin xyz="0.265391 0.32 -0.265" rpy="0 0 0"/>
     <geometry>
-      <mesh filename="$(find model_description)/meshes/r_caster_1.stl" scale="0.001 0.001 0.001"/>
+      <mesh filename="package://model_description/meshes/r_caster_1.stl" scale="0.001 0.001 0.001"/>
     </geometry>
     <material name="silver"/>
@@ -87,5 +87,5 @@
     <origin xyz="0.265391 0.32 -0.265" rpy="0 0 0"/>
     <geometry>
-      <mesh filename="$(find model_description)/meshes/r_caster_1.stl" scale="0.001 0.001 0.001"/>
+      <mesh filename="package://model_description/meshes/r_caster_1.stl" scale="0.001 0.001 0.001"/>
     </geometry>
   </collision>
@@ -100,5 +100,5 @@
     <origin xyz="0.27 -0.32 -0.265" rpy="0 0 0"/>
     <geometry>
-      <mesh filename="$(find model_description)/meshes/l_caster_1.stl" scale="0.001 0.001 0.001"/>
+      <mesh filename="package://model_description/meshes/l_caster_1.stl" scale="0.001 0.001 0.001"/>
     </geometry>
     <material name="silver"/>
@@ -107,5 +107,5 @@
     <origin xyz="0.27 -0.32 -0.265" rpy="0 0 0"/>
     <geometry>
-      <mesh filename="$(find model_description)/meshes/l_caster_1.stl" scale="0.001 0.001 0.001"/>
+      <mesh filename="package://model_description/meshes/l_caster_1.stl" scale="0.001 0.001 0.001"/>
     </geometry>
   </collision>
@@ -120,5 +120,5 @@
     <origin xyz="0.275391 0.35 -0.08" rpy="0 0 0"/>
     <geometry>
-      <mesh filename="$(find model_description)/meshes/r_caster_wheel_1.stl" scale="0.001 0.001 0.001"/>
+      <mesh filename="package://model_description/meshes/r_caster_wheel_1.stl" scale="0.001 0.001 0.001"/>
     </geometry>
     <material name="silver"/>
@@ -127,5 +127,5 @@
     <origin xyz="0.275391 0.35 -0.08" rpy="0 0 0"/>
     <geometry>
-      <mesh filename="$(find model_description)/meshes/r_caster_wheel_1.stl" scale="0.001 0.001 0.001"/>
+      <mesh filename="package://model_description/meshes/r_caster_wheel_1.stl" scale="0.001 0.001 0.001"/>
     </geometry>
   </collision>
@@ -140,5 +140,5 @@
     <origin xyz="0.28 -0.29 -0.08" rpy="0 0 0"/>
     <geometry>
-      <mesh filename="$(find model_description)/meshes/l_caster_wheel_1.stl" scale="0.001 0.001 0.001"/>
+      <mesh filename="package://model_description/meshes/l_caster_wheel_1.stl" scale="0.001 0.001 0.001"/>
     </geometry>
     <material name="silver"/>
@@ -147,5 +147,5 @@
     <origin xyz="0.28 -0.29 -0.08" rpy="0 0 0"/>
     <geometry>
-      <mesh filename="$(find model_description)/meshes/l_caster_wheel_1.stl" scale="0.001 0.001 0.001"/>
+      <mesh filename="package://model_description/meshes/l_caster_wheel_1.stl" scale="0.001 0.001 0.001"/>
     </geometry>
   </collision>
@@ -160,5 +160,5 @@
     <origin xyz="-1.14 0.34 -0.027" rpy="0 0 0"/>
     <geometry>
-      <mesh filename="$(find model_description)/meshes/r_static_wheel_1.stl" scale="0.001 0.001 0.001"/>
+      <mesh filename="package://model_description/meshes/r_static_wheel_1.stl" scale="0.001 0.001 0.001"/>
     </geometry>
     <material name="silver"/>
@@ -167,5 +167,5 @@
     <origin xyz="-1.14 0.34 -0.027" rpy="0 0 0"/>
     <geometry>
-      <mesh filename="$(find model_description)/meshes/r_static_wheel_1.stl" scale="0.001 0.001 0.001"/>
+      <mesh filename="package://model_description/meshes/r_static_wheel_1.stl" scale="0.001 0.001 0.001"/>
     </geometry>
   </collision>
@@ -180,5 +180,5 @@
     <origin xyz="-1.14 -0.34 -0.027" rpy="0 0 0"/>
     <geometry>
-      <mesh filename="$(find model_description)/meshes/l_static_wheel_1.stl" scale="0.001 0.001 0.001"/>
+      <mesh filename="package://model_description/meshes/l_static_wheel_1.stl" scale="0.001 0.001 0.001"/>
     </geometry>
     <material name="silver"/>
@@ -187,5 +187,5 @@
     <origin xyz="-1.14 -0.34 -0.027" rpy="0 0 0"/>
     <geometry>
-      <mesh filename="$(find model_description)/meshes/l_static_wheel_1.stl" scale="0.001 0.001 0.001"/>
+      <mesh filename="package://model_description/meshes/l_static_wheel_1.stl" scale="0.001 0.001 0.001"/>
     </geometry>
   </collision>
@@ -200,14 +200,14 @@
     <origin xyz="0.05 -0.29 -1.035" rpy="0 0 0"/>
     <geometry>
-      <mesh filename="$(find model_description)/meshes/steer_head_1.stl" scale="0.001 0.001 0.001"/>
-    </geometry>
-    <material name="silver"/>
-  </visual>
-  <collision>
+      <mesh filename="package://model_description/meshes/steer_head_1.stl" scale="0.001 0.001 0.001"/>
+    </geometry>
+    <material name="silver"/>
+  </visual>
+  <!-- <collision>
     <origin xyz="0.05 -0.29 -1.035" rpy="0 0 0"/>
     <geometry>
-      <mesh filename="$(find model_description)/meshes/steer_head_1.stl" scale="0.001 0.001 0.001"/>
-    </geometry>
-  </collision>
+      <mesh filename="package://model_description/meshes/steer_head_1.stl" scale="0.001 0.001 0.001"/>
+    </geometry>
+  </collision> -->
 </link>
 <link name="l_wheel_1">
@@ -220,5 +220,5 @@
     <origin xyz="0.902 0.345 -0.225194" rpy="0 0 0"/>
     <geometry>
-      <mesh filename="$(find model_description)/meshes/l_wheel_1.stl" scale="0.001 0.001 0.001"/>
+      <mesh filename="package://model_description/meshes/l_wheel_1.stl" scale="0.001 0.001 0.001"/>
     </geometry>
     <material name="silver"/>
@@ -227,5 +227,5 @@
     <origin xyz="0.902 0.345 -0.225194" rpy="0 0 0"/>
     <geometry>
-      <mesh filename="$(find model_description)/meshes/l_wheel_1.stl" scale="0.001 0.001 0.001"/>
+      <mesh filename="package://model_description/meshes/l_wheel_1.stl" scale="0.001 0.001 0.001"/>
     </geometry>
   </collision>
@@ -240,5 +240,5 @@
     <origin xyz="0.902 -0.345 -0.225194" rpy="0 0 0"/>
     <geometry>
-      <mesh filename="$(find model_description)/meshes/r_wheel_1.stl" scale="0.001 0.001 0.001"/>
+      <mesh filename="package://model_description/meshes/r_wheel_1.stl" scale="0.001 0.001 0.001"/>
     </geometry>
     <material name="silver"/>
@@ -247,5 +247,5 @@
     <origin xyz="0.902 -0.345 -0.225194" rpy="0 0 0"/>
     <geometry>
-      <mesh filename="$(find model_description)/meshes/r_wheel_1.stl" scale="0.001 0.001 0.001"/>
+      <mesh filename="package://model_description/meshes/r_wheel_1.stl" scale="0.001 0.001 0.001"/>
     </geometry>
   </collision>
@@ -260,14 +260,14 @@
     <origin xyz="0.902 -0.0 -0.533053" rpy="0 0 0"/>
     <geometry>
-      <mesh filename="$(find model_description)/meshes/steering_1.stl" scale="0.001 0.001 0.001"/>
-    </geometry>
-    <material name="silver"/>
-  </visual>
-  <collision>
+      <mesh filename="package://model_description/meshes/steering_1.stl" scale="0.001 0.001 0.001"/>
+    </geometry>
+    <material name="silver"/>
+  </visual>
+  <!-- <collision>
     <origin xyz="0.902 -0.0 -0.533053" rpy="0 0 0"/>
     <geometry>
-      <mesh filename="$(find model_description)/meshes/steering_1.stl" scale="0.001 0.001 0.001"/>
-    </geometry>
-  </collision>
+      <mesh filename="package://model_description/meshes/steering_1.stl" scale="0.001 0.001 0.001"/>
+    </geometry>
+  </collision> -->
 </link>
 <link name="camera_link">
@@ -360,6 +360,7 @@
   <parent link="steer_head_1"/>
   <child link="steering_1"/>
-  <axis xyz="-0.0 -0.0 1.0"/>
-  <limit upper="-0.7853982" lower="0.7853982" effort="100" velocity="100"/>
+  <axis xyz="0 0 1"/>
+  <limit upper="0.785398163" lower="-0.785398163" effort="100" velocity="3"/>
+  <dynamics damping="0.1"/>
 </joint>
 <!-- custom joint for sensors -->
