Commit message: replacing ascamera lib'

File: src/ddmr_description/urdf/ddmr.xacro (robot description, xacro)
@@ -4,4 +4,10 @@
   <xacro:include filename="$(find ddmr_description)/urdf/ddmr.ros2control" />
   <xacro:include filename="$(find ddmr_description)/urdf/ddmr.gazebo" />
+  <link name="base_footprint"></link>
+  <joint name="base_joint" type="fixed">
+    <parent link="base_footprint"/>
+    <child link="base_link"/>
+    <origin xyz="0.0 0.0 0.010" rpy="0 0 0"/>
+  </joint>
   <link name="base_link">
     <inertial>
@@ -34,5 +40,5 @@
     </collision>
   </link>
-  <link name="rwheel_1">
+  <link name="rwheel">
     <inertial>
       <origin xyz="0.0 0.01575 0.0" rpy="0 0 0"/>
@@ -52,5 +58,5 @@
       <geometry>
         <mesh
-          filename="file://$(find ddmr_description)/meshes/rwheel_1.stl"
+          filename="file://$(find ddmr_description)/meshes/rwheel.stl"
           scale="0.001 0.001 0.001"/>
       </geometry>
@@ -63,10 +69,10 @@
       <geometry>
         <mesh
-          filename="file://$(find ddmr_description)/meshes/rwheel_1.stl"
+          filename="file://$(find ddmr_description)/meshes/rwheel.stl"
           scale="0.001 0.001 0.001"/>
       </geometry>
     </collision>
   </link>
-  <link name="lwheel_1">
+  <link name="lwheel">
     <inertial>
       <origin xyz="0.0 -0.01575 0.0" rpy="0 0 0"/>
@@ -86,5 +92,5 @@
       <geometry>
         <mesh
-          filename="file://$(find ddmr_description)/meshes/lwheel_1.stl"
+          filename="file://$(find ddmr_description)/meshes/lwheel.stl"
           scale="0.001 0.001 0.001"/>
       </geometry>
@@ -97,10 +103,10 @@
       <geometry>
         <mesh
-          filename="file://$(find ddmr_description)/meshes/lwheel_1.stl"
+          filename="file://$(find ddmr_description)/meshes/lwheel.stl"
           scale="0.001 0.001 0.001"/>
       </geometry>
     </collision>
   </link>
-  <link name="camera_1">
+  <link name="camera">
     <inertial>
       <origin xyz="0.0 0.0 0.0095" rpy="0 0 0"/>
@@ -120,5 +126,5 @@
       <geometry>
         <mesh
-          filename="file://$(find ddmr_description)/meshes/camera_1.stl"
+          filename="file://$(find ddmr_description)/meshes/camera.stl"
           scale="0.001 0.001 0.001"/>
       </geometry>
@@ -131,5 +137,5 @@
       <geometry>
         <mesh
-          filename="file://$(find ddmr_description)/meshes/camera_1.stl"
+          filename="file://$(find ddmr_description)/meshes/camera.stl"
           scale="0.001 0.001 0.001"/>
       </geometry>
@@ -141,5 +147,5 @@
       rpy="0 0 0"/>
     <parent link="base_link"/>
-    <child link="rwheel_1"/>
+    <child link="rwheel"/>
     <!-- Wheel axle is now Y -->
     <axis xyz="0 1 0"/>
@@ -150,5 +156,5 @@
       rpy="0 0 0"/>
     <parent link="base_link"/>
-    <child link="lwheel_1"/>
+    <child link="lwheel"/>
     <!-- Wheel axle is now Y -->
     <axis xyz="0 -1 0"/>
@@ -159,5 +165,5 @@
       rpy="0 0 0"/>
     <parent link="base_link"/>
-    <child link="camera_1"/>
+    <child link="camera"/>
   </joint>
 </robot>

Commit message: backup slam

File: src/ddmr_description/urdf/ddmr.xacro (robot description, xacro)
@@ -108,5 +108,5 @@
     </collision>
   </link>
-  <link name="camera">
+  <link name="camera_link">
     <inertial>
       <origin xyz="0.0 0.0 0.0095" rpy="0 0 0"/>
@@ -126,5 +126,5 @@
       <geometry>
         <mesh
-          filename="file://$(find ddmr_description)/meshes/camera.stl"
+          filename="file://$(find ddmr_description)/meshes/camera_link.stl"
           scale="0.001 0.001 0.001"/>
       </geometry>
@@ -137,5 +137,5 @@
       <geometry>
         <mesh
-          filename="file://$(find ddmr_description)/meshes/camera.stl"
+          filename="file://$(find ddmr_description)/meshes/camera_link.stl"
           scale="0.001 0.001 0.001"/>
       </geometry>
@@ -165,5 +165,5 @@
       rpy="0 0 0"/>
     <parent link="base_link"/>
-    <child link="camera"/>
+    <child link="camera_link"/>
   </joint>
 </robot>
