Commit message: working on tracker

File: src/agv_description/urdf/model.xacro (robot description, xacro)
@@ -4,248 +4,22 @@
 <xacro:include filename="$(find agv_description)/urdf/model.ros2control" />
 <xacro:include filename="$(find agv_description)/urdf/model.gazebo" />
-<xacro:include filename="$(find agv_description)/urdf/camera.xacro" />
-<link name="base_footprint"></link>
-<joint name="base_joint" type="fixed">
-  <parent link="base_footprint"/>
-  <child link="base_link"/>
-  <origin xyz="0.0 0.0 0.010" rpy="0 0 0"/>
-</joint>
+<xacro:include filename="$(find agv_description)/urdf/sensors.xacro" />
 <link name="base_link">
   <inertial>
-    <origin xyz="0.058268932725645046 5.2977171567329385e-05 0.727540488639707" rpy="0 0 0"/>
-    <mass value="17.8126449840257"/>
-    <inertia ixx="6.934301" iyy="7.211008" izz="2.123225" ixy="0.000338" iyz="0.00046" ixz="1.178057"/>
+    <origin xyz="0.1595846051428766 0.001628061693118389 0.3212324983015764" rpy="0 0 0"/>
+    <mass value="74.92687542221871"/>
+    <inertia ixx="11.521815" iyy="13.012549" izz="19.198561" ixy="-0.104416" iyz="-0.011996" ixz="-0.669571"/>
   </inertial>
   <visual>
     <origin xyz="0 0 0" rpy="0 0 0"/>
     <geometry>
-      <mesh filename="package://agv_description/meshes/base_link.stl" scale="0.001 0.001 0.001"/>
-    </geometry>
-    <material name="silver"/>
-  </visual>
-  <!-- <collision>
+      <mesh filename="file://$(find agv_description)/meshes/base_link.stl" scale="0.001 0.001 0.001"/>
+    </geometry>
+    <material name="silver"/>
+  </visual>
+  <collision>
     <origin xyz="0 0 0" rpy="0 0 0"/>
     <geometry>
-      <mesh filename="package://agv_description/meshes/base_link.stl" scale="0.001 0.001 0.001"/>
-    </geometry>
-  </collision> -->
-</link>
-<link name="stacker_slider_1">
-  <inertial>
-    <origin xyz="-0.013466560993404583 0.2572823159739083 -1.6689840557999553" rpy="0 0 0"/>
-    <mass value="2.158204417874895"/>
-    <inertia ixx="0.17152" iyy="0.054313" izz="0.126927" ixy="-3.9e-05" iyz="-0.000468" ixz="-0.00104"/>
-  </inertial>
-  <visual>
-    <origin xyz="-0.05 0.256 -1.99" rpy="0 0 0"/>
-    <geometry>
-      <mesh filename="package://agv_description/meshes/stacker_slider_1.stl" scale="0.001 0.001 0.001"/>
-    </geometry>
-    <material name="silver"/>
-  </visual>
-  <collision>
-    <origin xyz="-0.05 0.256 -1.99" rpy="0 0 0"/>
-    <geometry>
-      <mesh filename="package://agv_description/meshes/stacker_slider_1.stl" scale="0.001 0.001 0.001"/>
-    </geometry>
-  </collision>
-</link>
-<link name="stacker_fork_1">
-  <inertial>
-    <origin xyz="0.09916634957104192 0.37114014282073293 -0.21646507194627185" rpy="0 0 0"/>
-    <mass value="8.37653098650869"/>
-    <inertia ixx="0.832862" iyy="0.734326" izz="1.204215" ixy="0.000947" iyz="-0.002067" ixz="0.159217"/>
-  </inertial>
-  <visual>
-    <origin xyz="-0.125 0.375 -0.49" rpy="0 0 0"/>
-    <geometry>
-      <mesh filename="package://agv_description/meshes/stacker_fork_1.stl" scale="0.001 0.001 0.001"/>
-    </geometry>
-    <material name="silver"/>
-  </visual>
-  <collision>
-    <origin xyz="-0.125 0.375 -0.49" rpy="0 0 0"/>
-    <geometry>
-      <mesh filename="package://agv_description/meshes/stacker_fork_1.stl" scale="0.001 0.001 0.001"/>
-    </geometry>
-  </collision>
-</link>
-<link name="r_caster_1">
-  <inertial>
-    <origin xyz="-0.005926729995574753 -6.024346577149231e-10 -0.08540642916490254" rpy="0 0 0"/>
-    <mass value="0.13643173338288486"/>
-    <inertia ixx="0.000369" iyy="0.000354" izz="9e-05" ixy="0.0" iyz="-0.0" ixz="-3.3e-05"/>
-  </inertial>
-  <visual>
-    <origin xyz="0.265391 0.32 -0.265" rpy="0 0 0"/>
-    <geometry>
-      <mesh filename="package://agv_description/meshes/r_caster_1.stl" scale="0.001 0.001 0.001"/>
-    </geometry>
-    <material name="silver"/>
-  </visual>
-  <collision>
-    <origin xyz="0.265391 0.32 -0.265" rpy="0 0 0"/>
-    <geometry>
-      <mesh filename="package://agv_description/meshes/r_caster_1.stl" scale="0.001 0.001 0.001"/>
-    </geometry>
-  </collision>
-</link>
-<link name="l_caster_1">
-  <inertial>
-    <origin xyz="-0.00592651973504249 -6.024346022037719e-10 -0.08540642916490221" rpy="0 0 0"/>
-    <mass value="0.13643173338288483"/>
-    <inertia ixx="0.000369" iyy="0.000354" izz="9e-05" ixy="0.0" iyz="-0.0" ixz="-3.3e-05"/>
-  </inertial>
-  <visual>
-    <origin xyz="0.27 -0.32 -0.265" rpy="0 0 0"/>
-    <geometry>
-      <mesh filename="package://agv_description/meshes/l_caster_1.stl" scale="0.001 0.001 0.001"/>
-    </geometry>
-    <material name="silver"/>
-  </visual>
-  <collision>
-    <origin xyz="0.27 -0.32 -0.265" rpy="0 0 0"/>
-    <geometry>
-      <mesh filename="package://agv_description/meshes/l_caster_1.stl" scale="0.001 0.001 0.001"/>
-    </geometry>
-  </collision>
-</link>
-<link name="r_caster_wheel_1">
-  <inertial>
-    <origin xyz="-2.1026053198536232e-07 0.03499999999999992 -9.71445146547012e-17" rpy="0 0 0"/>
-    <mass value="0.9633599527692169"/>
-    <inertia ixx="0.002258" iyy="0.004173" izz="0.002258" ixy="-0.0" iyz="-0.0" ixz="0.0"/>
-  </inertial>
-  <visual>
-    <origin xyz="0.275391 0.35 -0.08" rpy="0 0 0"/>
-    <geometry>
-      <mesh filename="package://agv_description/meshes/r_caster_wheel_1.stl" scale="0.001 0.001 0.001"/>
-    </geometry>
-    <material name="silver"/>
-  </visual>
-  <collision>
-    <origin xyz="0.275391 0.35 -0.08" rpy="0 0 0"/>
-    <geometry>
-      <mesh filename="package://agv_description/meshes/r_caster_wheel_1.stl" scale="0.001 0.001 0.001"/>
-    </geometry>
-  </collision>
-</link>
-<link name="l_caster_wheel_1">
-  <inertial>
-    <origin xyz="5.551115123125783e-17 0.03500000000000003 4.3021142204224816e-16" rpy="0 0 0"/>
-    <mass value="0.9633599527692169"/>
-    <inertia ixx="0.002258" iyy="0.004173" izz="0.002258" ixy="0.0" iyz="0.0" ixz="0.0"/>
-  </inertial>
-  <visual>
-    <origin xyz="0.28 -0.29 -0.08" rpy="0 0 0"/>
-    <geometry>
-      <mesh filename="package://agv_description/meshes/l_caster_wheel_1.stl" scale="0.001 0.001 0.001"/>
-    </geometry>
-    <material name="silver"/>
-  </visual>
-  <collision>
-    <origin xyz="0.28 -0.29 -0.08" rpy="0 0 0"/>
-    <geometry>
-      <mesh filename="package://agv_description/meshes/l_caster_wheel_1.stl" scale="0.001 0.001 0.001"/>
-    </geometry>
-  </collision>
-</link>
-<link name="r_static_wheel_1">
-  <inertial>
-    <origin xyz="-2.220446049250313e-16 0.04999999999999977 -1.0061396160665481e-16" rpy="0 0 0"/>
-    <mass value="0.322264574405241"/>
-    <inertia ixx="0.000266" iyy="0.000208" izz="0.000266" ixy="0.0" iyz="0.0" ixz="0.0"/>
-  </inertial>
-  <visual>
-    <origin xyz="-1.14 0.34 -0.027" rpy="0 0 0"/>
-    <geometry>
-      <mesh filename="package://agv_description/meshes/r_static_wheel_1.stl" scale="0.001 0.001 0.001"/>
-    </geometry>
-    <material name="silver"/>
-  </visual>
-  <collision>
-    <origin xyz="-1.14 0.34 -0.027" rpy="0 0 0"/>
-    <geometry>
-      <mesh filename="package://agv_description/meshes/r_static_wheel_1.stl" scale="0.001 0.001 0.001"/>
-    </geometry>
-  </collision>
-</link>
-<link name="l_static_wheel_1">
-  <inertial>
-    <origin xyz="-2.220446049250313e-16 -0.050000000000000544 -1.2836953722228372e-16" rpy="0 0 0"/>
-    <mass value="0.322264574405241"/>
-    <inertia ixx="0.000266" iyy="0.000208" izz="0.000266" ixy="0.0" iyz="0.0" ixz="0.0"/>
-  </inertial>
-  <visual>
-    <origin xyz="-1.14 -0.34 -0.027" rpy="0 0 0"/>
-    <geometry>
-      <mesh filename="package://agv_description/meshes/l_static_wheel_1.stl" scale="0.001 0.001 0.001"/>
-    </geometry>
-    <material name="silver"/>
-  </visual>
-  <collision>
-    <origin xyz="-1.14 -0.34 -0.027" rpy="0 0 0"/>
-    <geometry>
-      <mesh filename="package://agv_description/meshes/l_static_wheel_1.stl" scale="0.001 0.001 0.001"/>
-    </geometry>
-  </collision>
-</link>
-<link name="steer_head_1">
-  <inertial>
-    <origin xyz="-0.5920522484243218 -0.29000000000059517 -0.3990675887191176" rpy="0 0 0"/>
-    <mass value="9.632954680220392"/>
-    <inertia ixx="0.447234" iyy="0.67858" izz="1.090345" ixy="0.0" iyz="-0.0" ixz="0.001718"/>
-  </inertial>
-  <visual>
-    <origin xyz="0.05 -0.29 -1.035" rpy="0 0 0"/>
-    <geometry>
-      <mesh filename="package://agv_description/meshes/steer_head_1.stl" scale="0.001 0.001 0.001"/>
-    </geometry>
-    <material name="silver"/>
-  </visual>
-  <!-- <collision>
-    <origin xyz="0.05 -0.29 -1.035" rpy="0 0 0"/>
-    <geometry>
-      <mesh filename="package://agv_description/meshes/steer_head_1.stl" scale="0.001 0.001 0.001"/>
-    </geometry>
-  </collision> -->
-</link>
-<link name="l_wheel_1">
-  <inertial>
-    <origin xyz="-3.975279472268056e-08 -0.0561204250420686 -2.6132590674743383e-08" rpy="0 0 0"/>
-    <mass value="8.335497772675197"/>
-    <inertia ixx="0.1042" iyy="0.188397" izz="0.1042" ixy="0.0" iyz="-0.0" ixz="-0.0"/>
-  </inertial>
-  <visual>
-    <origin xyz="0.902 0.345 -0.225194" rpy="0 0 0"/>
-    <geometry>
-      <mesh filename="package://agv_description/meshes/l_wheel_1.stl" scale="0.001 0.001 0.001"/>
-    </geometry>
-    <material name="silver"/>
-  </visual>
-  <collision>
-    <origin xyz="0.902 0.345 -0.225194" rpy="0 0 0"/>
-    <geometry>
-      <mesh filename="package://agv_description/meshes/l_wheel_1.stl" scale="0.001 0.001 0.001"/>
-    </geometry>
-  </collision>
-</link>
-<link name="r_wheel_1">
-  <inertial>
-    <origin xyz="3.975264217803698e-08 0.0561204250421648 -2.6132589647787086e-08" rpy="0 0 0"/>
-    <mass value="8.335497772675197"/>
-    <inertia ixx="0.1042" iyy="0.188397" izz="0.1042" ixy="0.0" iyz="0.0" ixz="0.0"/>
-  </inertial>
-  <visual>
-    <origin xyz="0.902 -0.345 -0.225194" rpy="0 0 0"/>
-    <geometry>
-      <mesh filename="package://agv_description/meshes/r_wheel_1.stl" scale="0.001 0.001 0.001"/>
-    </geometry>
-    <material name="silver"/>
-  </visual>
-  <collision>
-    <origin xyz="0.902 -0.345 -0.225194" rpy="0 0 0"/>
-    <geometry>
-      <mesh filename="package://agv_description/meshes/r_wheel_1.stl" scale="0.001 0.001 0.001"/>
+      <mesh filename="file://$(find agv_description)/meshes/base_link.stl" scale="0.001 0.001 0.001"/>
     </geometry>
   </collision>
@@ -253,23 +27,143 @@
 <link name="steering_1">
   <inertial>
-    <origin xyz="0.000175198957576006 -0.026843466909504198 -0.2259057384340462" rpy="0 0 0"/>
-    <mass value="7.502979344444109"/>
-    <inertia ixx="0.248967" iyy="0.21124" izz="0.32283" ixy="0.000231" iyz="0.002116" ixz="0.001067"/>
-  </inertial>
-  <visual>
-    <origin xyz="0.902 -0.0 -0.533053" rpy="0 0 0"/>
-    <geometry>
-      <mesh filename="package://agv_description/meshes/steering_1.stl" scale="0.001 0.001 0.001"/>
-    </geometry>
-    <material name="silver"/>
-  </visual>
-  <!-- <collision>
-    <origin xyz="0.902 -0.0 -0.533053" rpy="0 0 0"/>
-    <geometry>
-      <mesh filename="package://agv_description/meshes/steering_1.stl" scale="0.001 0.001 0.001"/>
-    </geometry>
-  </collision> -->
-</link>
-<link name="camera_link">
+    <origin xyz="-0.0002292488980326907 -0.03933024782494826 -0.17867777408636726" rpy="0 0 0"/>
+    <mass value="76.54947604055778"/>
+    <inertia ixx="3.654942" iyy="2.105298" izz="4.532864" ixy="-0.033032" iyz="-0.01099" ixz="0.024409"/>
+  </inertial>
+  <visual>
+    <origin xyz="0.0 -0.0 0.0" rpy="0 0 0"/>
+    <geometry>
+      <mesh filename="file://$(find agv_description)/meshes/steering_1.stl" scale="0.001 0.001 0.001"/>
+    </geometry>
+    <material name="silver"/>
+  </visual>
+  <collision>
+    <origin xyz="0.0 -0.0 0.0" rpy="0 0 0"/>
+    <geometry>
+      <mesh filename="file://$(find agv_description)/meshes/steering_1.stl" scale="0.001 0.001 0.001"/>
+    </geometry>
+  </collision>
+</link>
+<link name="rr_wheel_1">
+  <inertial>
+    <origin xyz="3.298326510048355e-07 -0.05488071442175224 -1.3094392831147772e-07" rpy="0 0 0"/>
+    <mass value="8.066605493230483"/>
+    <inertia ixx="0.102004" iyy="0.184234" izz="0.102004" ixy="0.0" iyz="-0.0" ixz="0.0"/>
+  </inertial>
+  <visual>
+    <origin xyz="-0.0 0.335 0.27" rpy="0 0 0"/>
+    <geometry>
+      <mesh filename="file://$(find agv_description)/meshes/rr_wheel_1.stl" scale="0.001 0.001 0.001"/>
+    </geometry>
+    <material name="silver"/>
+  </visual>
+  <collision>
+    <origin xyz="-0.0 0.335 0.27" rpy="0 0 0"/>
+    <geometry>
+      <mesh filename="file://$(find agv_description)/meshes/rr_wheel_1.stl" scale="0.001 0.001 0.001"/>
+    </geometry>
+  </collision>
+</link>
+<link name="lr_wheel_1">
+  <inertial>
+    <origin xyz="-6.410595517536421e-08 0.054880694868648994 -4.107795414931559e-08" rpy="0 0 0"/>
+    <mass value="8.066582577854387"/>
+    <inertia ixx="0.102003" iyy="0.184233" izz="0.102003" ixy="0.0" iyz="-0.0" ixz="-0.0"/>
+  </inertial>
+  <visual>
+    <origin xyz="-0.0 -0.335 0.27" rpy="0 0 0"/>
+    <geometry>
+      <mesh filename="file://$(find agv_description)/meshes/lr_wheel_1.stl" scale="0.001 0.001 0.001"/>
+    </geometry>
+    <material name="silver"/>
+  </visual>
+  <collision>
+    <origin xyz="-0.0 -0.335 0.27" rpy="0 0 0"/>
+    <geometry>
+      <mesh filename="file://$(find agv_description)/meshes/lr_wheel_1.stl" scale="0.001 0.001 0.001"/>
+    </geometry>
+  </collision>
+</link>
+<link name="stacker_1">
+  <inertial>
+    <origin xyz="0.1667105127366031 0.2899679742039218 -0.20090477981280133" rpy="0 0 0"/>
+    <mass value="114.38554635922912"/>
+    <inertia ixx="43.717987" iyy="40.031482" izz="16.275385" ixy="-0.000734" iyz="0.001845" ixz="5.713124"/>
+  </inertial>
+  <visual>
+    <origin xyz="-0.849999 0.290502 -0.114" rpy="0 0 0"/>
+    <geometry>
+      <mesh filename="file://$(find agv_description)/meshes/stacker_1.stl" scale="0.001 0.001 0.001"/>
+    </geometry>
+    <material name="silver"/>
+  </visual>
+  <collision>
+    <origin xyz="-0.849999 0.290502 -0.114" rpy="0 0 0"/>
+    <geometry>
+      <mesh filename="file://$(find agv_description)/meshes/stacker_1.stl" scale="0.001 0.001 0.001"/>
+    </geometry>
+  </collision>
+</link>
+<link name="rf_wheel_1">
+  <inertial>
+    <origin xyz="4.713639616404919e-07 0.03000045322132716 5.773159728050814e-15" rpy="0 0 0"/>
+    <mass value="0.29853713005801513"/>
+    <inertia ixx="0.000202" iyy="0.000278" izz="0.000202" ixy="0.0" iyz="-0.0" ixz="0.0"/>
+  </inertial>
+  <visual>
+    <origin xyz="-1.659999 0.350502 0.4615" rpy="0 0 0"/>
+    <geometry>
+      <mesh filename="file://$(find agv_description)/meshes/rf_wheel_1.stl" scale="0.001 0.001 0.001"/>
+    </geometry>
+    <material name="silver"/>
+  </visual>
+  <collision>
+    <origin xyz="-1.659999 0.350502 0.4615" rpy="0 0 0"/>
+    <geometry>
+      <mesh filename="file://$(find agv_description)/meshes/rf_wheel_1.stl" scale="0.001 0.001 0.001"/>
+    </geometry>
+  </collision>
+</link>
+<link name="lf_wheel_1">
+  <inertial>
+    <origin xyz="4.7136395964209044e-07 0.030000453221327716 8.049116928532385e-15" rpy="0 0 0"/>
+    <mass value="0.29853713005801513"/>
+    <inertia ixx="0.000202" iyy="0.000278" izz="0.000202" ixy="-0.0" iyz="0.0" ixz="0.0"/>
+  </inertial>
+  <visual>
+    <origin xyz="-1.659999 -0.289498 0.4615" rpy="0 0 0"/>
+    <geometry>
+      <mesh filename="file://$(find agv_description)/meshes/lf_wheel_1.stl" scale="0.001 0.001 0.001"/>
+    </geometry>
+    <material name="silver"/>
+  </visual>
+  <collision>
+    <origin xyz="-1.659999 -0.289498 0.4615" rpy="0 0 0"/>
+    <geometry>
+      <mesh filename="file://$(find agv_description)/meshes/lf_wheel_1.stl" scale="0.001 0.001 0.001"/>
+    </geometry>
+  </collision>
+</link>
+<link name="fork_1">
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
Commit message: workin on laster merge

File: src/agv_description/urdf/model.xacro (robot description, xacro)
@@ -165,5 +165,45 @@
   </collision>
 </link>
-<link name="front_lidar_link">
+<link name="left_lidar_link">
+  <inertial>
+    <origin xyz="0.0 0.0 0.0" rpy="0 0 0"/>
+    <mass value="0.1"/>
+    <inertia ixx="0.0001" iyy="0.0001" izz="0.0001" ixy="0.0" iyz="0.0" ixz="0.0"/>
+  </inertial>
+  <visual>
+    <origin xyz="0.0 0.0 0.0" rpy="0 0 0"/>
+    <geometry>
+      <cylinder radius="0.03" length="0.012"/>
+    </geometry>
+    <material name="red"/>
+  </visual>
+  <collision>
+    <origin xyz="0.0 0.0 0.0" rpy="0 0 0"/>
+    <geometry>
+      <cylinder radius="0.03" length="0.012"/>
+    </geometry>
+  </collision>
+</link>
+<link name="right_lidar_link">
+  <inertial>
+    <origin xyz="0.0 0.0 0.0" rpy="0 0 0"/>
+    <mass value="0.1"/>
+    <inertia ixx="0.0001" iyy="0.0001" izz="0.0001" ixy="0.0" iyz="0.0" ixz="0.0"/>
+  </inertial>
+  <visual>
+    <origin xyz="0.0 0.0 0.0" rpy="0 0 0"/>
+    <geometry>
+      <cylinder radius="0.03" length="0.012"/>
+    </geometry>
+    <material name="red"/>
+  </visual>
+  <collision>
+    <origin xyz="0.0 0.0 0.0" rpy="0 0 0"/>
+    <geometry>
+      <cylinder radius="0.03" length="0.012"/>
+    </geometry>
+  </collision>
+</link>
+<link name="merge_lidar_link">
   <inertial>
     <origin xyz="0.0 0.0 0.0" rpy="0 0 0"/>
@@ -228,8 +268,18 @@
   <limit upper="1.2" lower="0.0" effort="100" velocity="100"/>
 </joint>
-<joint name="front_lidar_joint" type="fixed">
+<joint name="left_lidar_joint" type="fixed">
   <origin xyz="0.8 0.4 -0.32" rpy="0 0 0"/>
   <parent link="base_link"/>
-  <child link="front_lidar_link"/>
+  <child link="left_lidar_link"/>
+</joint>
+<joint name="right_lidar_joint" type="fixed">
+  <origin xyz="0.8 -0.4 -0.32" rpy="0 0 0"/>
+  <parent link="base_link"/>
+  <child link="right_lidar_link"/>
+</joint>
+<joint name="merge_lidar_joint" type="fixed">
+  <origin xyz="0.0 0.0 -0.32" rpy="0 0 0"/>
+  <parent link="base_link"/>
+  <child link="merge_lidar_link"/>
 </joint>
 </robot>

File: src/agv_description/urdf/sensors.xacro (robot description, xacro)
@@ -1,6 +1,30 @@
 <?xml version="1.0"?>
 <robot name="model" xmlns:xacro="http://www.ros.org/wiki/xacro">
-  <gazebo reference="front_lidar_link">
-    <sensor name="front_lidar" type="gpu_lidar">
+  <gazebo reference="left_lidar_link">
+    <sensor name="left_lidar" type="gpu_lidar">
+      <pose>0 0 0 0 0 0</pose>
+      <always_on>true</always_on>
+      <visualize>true</visualize>
+      <update_rate>10</update_rate>
+      <topic>/scan</topic>
+      <lidar>
+        <scan>
+          <horizontal>
+            <samples>720</samples>
+            <resolution>1</resolution>
+            <min_angle>-3.14159</min_angle>
+            <max_angle>3.14159</max_angle>
+          </horizontal>
+        </scan>
+        <range>
+          <min>0.10</min>
+          <max>30.0</max>
+          <resolution>0.01</resolution>
+        </range>
+      </lidar>
+    </sensor>
+  </gazebo>
+  <gazebo reference="right_lidar_link">
+    <sensor name="right_lidar" type="gpu_lidar">
       <pose>0 0 0 0 0 0</pose>
       <always_on>true</always_on>
